File: PCB/hotswap_choc/helix.kicad_pcb (KiCad board)
At the start: 2 copper layers, 135.2 x 94 mm, 134 parts, among them J1 MJ-4PP-9, P1 CONN_01X01, P2 CONN_01X01, P3 OLED, P4 LED, SW1 SW_PUSH, SW10 SW_PUSH, SW11 SW_PUSH, SW12 SW_PUSH, SW13 SW_PUSH, SW14 SW_PUSH, SW15 SW_PUSH, SW16 SW_PUSH, SW17 SW_PUSH, SW18 SW_PUSH, SW19 SW_PUSH, SW2 SW_PUSH, SW20 SW_PUSH, SW21 SW_PUSH, SW22 SW_PUSH, SW23 SW_PUSH, SW24 SW_PUSH, SW25 SW_PUSH, SW26 SW_PUSH, SW27 SW_PUSH, SW28 SW_PUSH, SW29 SW_PUSH, SW3 SW_PUSH, SW30 SW_PUSH, SW31 SW_PUSH, SW32 SW_PUSH, SW33 Reset, SW4 SW_PUSH, SW5 SW_PUSH, SW6 SW_PUSH, SW7 SW_PUSH, SW8 SW_PUSH, SW9 SW_PUSH, U1 ProMicro, U10 SK6812mini, U11 SK6812mini, U12 SK6812mini, U13 SK6812mini, U14 SK6812mini, U15 SK6812mini, U16 SK6812mini, U17 SK6812mini, U18 SK6812mini, U19 SK6812mini, U2 SK6812mini, U20 SK6812mini, U21 SK6812mini, U22 SK6812mini, U23 SK6812mini, U24 SK6812mini, U25 SK6812mini, U26 SK6812mini, U27 SK6812mini, U28 SK6812mini, U29 SK6812mini, U3 SK6812mini, U30 SK6812mini, U31 SK6812mini, U32 SK6812mini, U33 SK6812mini, U4 SK6812mini, U5 SK6812mini, U6 SK6812mini, U7 SK6812mini, U8 SK6812mini, U9 SK6812mini

Commit message: Update
Parts:
- moved D24 13.8 mm to (178.7, 108.5), turned to 270 degrees
- moved D19 13.8 mm to (83.7, 108.5), turned to 270 degrees
- moved D20 13.8 mm to (102.7, 108.5), turned to 270 degrees
- moved D21 13.8 mm to (121.7, 108.5), turned to 270 degrees
- moved D22 13.8 mm to (140.7, 108.5), turned to 270 degrees
- moved D23 13.8 mm to (159.7, 108.5), turned to 270 degrees
- moved D25 13.8 mm to (197.7, 108.5), turned to 270 degrees
Routing:
- net row4: track 246.2 -> 218.2 mm, vias 11 -> 17
- net row3: track 199.9 -> 188.3 mm, vias 10 -> 15
- net VCC: track 1047.3 -> 1057.6 mm, vias 41 -> 43
- net Net-(D19-Pad2): track 32.7 -> 23.5 mm
- net GND: track 919.6 -> 928.5 mm
- net Net-(D24-Pad2): track 31.1 -> 23.5 mm
- net Net-(D20-Pad2): track 31.0 -> 23.5 mm
- net Net-(D21-Pad2): track 31.0 -> 23.5 mm
- net Net-(D22-Pad2): track 31.0 -> 23.5 mm
- net Net-(D25-Pad2): track 31.0 -> 23.5 mm
- net Net-(D23-Pad2): track 31.0 -> 23.5 mm
- net col1: track 256.5 -> 263.9 mm, vias 7 -> 5
- net col2: track 225.7 -> 233.1 mm, vias 10 -> 8
- net col4: track 179.2 -> 186.5 mm, vias 8 -> 6
- net col0: track 296.4 -> 301.6 mm, vias 9 -> 7
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Other:
- outline, holes or cut-outs redrawn
